Commit message: scara_2limb

File: 3D models/scara2/exports/assembly.SLDASM/urdf/assembly.SLDASM.urdf (robot description, URDF)
Before this commit: robot assembly.SLDASM, 3 links, 2 joints
Joints:
- joint joint1: limit lower=-1.57 upper=1.57 effort=0 velocity=0 -> lower=-0.7854 upper=0.7854 effort=0 velocity=0; origin xyz=0 0 0.075 rpy=1.5708 0 -1.1781 -> xyz=0 0 0.075 rpy=1.5708 0 0
- joint joint2: limit lower=-1.57 upper=1.57 effort=0 velocity=0 -> lower=-0.7854 upper=0.7854 effort=0 velocity=0; origin xyz=0.2 0 0 rpy=0 0.98163 0 -> xyz=0.2 0 0 rpy=0 0 0

Commit message: scara fix

File: 3D models/scara2/exports/assembly.SLDASM/urdf/assembly.SLDASM.urdf (robot description, URDF)
Before this commit: robot assembly.SLDASM, 3 links, 2 joints
Joints:
- joint joint1: limit lower=-0.7854 upper=0.7854 effort=0 velocity=0 -> lower=-1.5708 upper=1.5708 effort=0 velocity=0
- joint joint2: limit lower=-0.7854 upper=0.7854 effort=0 velocity=0 -> lower=-1.5708 upper=1.5708 effort=0 velocity=0
